File: PCB/AstralCNC.kicad_sch (KiCad schematic)
At the start: 47 parts, among them J1 USB_C_Receptacle_USB2.0_16P, J11 Conn_01x02, J31 Conn_01x10_Pin, J310 Conn_02x04_Counter_Clockwise, J311 Conn_01x04_Pin, J312 Conn_01x04_Pin, J313 Conn_01x04_Pin, J32 Conn_01x04_Pin, J33 Conn_01x03_Pin, J34 Conn_01x03_Pin, J35 Conn_01x03_Pin, J36 Conn_01x03_Pin, J37 Conn_01x04_Pin, J38 Conn_01x04_Pin, J39 Conn_01x04_Pin, Q21 BC847, Q22 BC847, Q23 BC847, U11 AP63357, U21 74HC244, U22 74HC244, U31 RP2350_Stamp, U32 TXS0108EPW, U33 TXS0108EPW

Commit message: bruh
Parts:
- added D1: LED, Connector_PinHeader_2.54mm:PinHeader_1x02_P2.54mm_Vertical, symbol Device:LED
- added D31: D_Shockley, Diode_SMD:D_SMA_Handsoldering, symbol Device:D_Shockley
- added R1: R, Capacitor_SMD:C_0603_1608Metric_Pad1.08x0.95mm_HandSolder, symbol Device:R
- J314: renamed from J1; footprint (none) -> Connector_USB:USB_C_Receptacle_G-Switch_GT-USB-7010ASV
- R31: renamed from R1; footprint (none) -> Capacitor_SMD:C_0603_1608Metric_Pad1.08x0.95mm_HandSolder
- R32: renamed from R2; footprint (none) -> Capacitor_SMD:C_0603_1608Metric_Pad1.08x0.95mm_HandSolder
Connections:
- net +5V: now also D31.1 (K)
- net AUX1: now also D1.2 (A); no longer J31.5 (Pin_5)
- net AUX2: now also J31.5 (Pin_5); no longer J31.4 (Pin_4)
- net AUX3: now also J31.4 (Pin_4); no longer J31.3 (Pin_3)
- net AUX_4: now also J31.3 (Pin_3)
- net GND: now also J314.A1 (GND), J314.A12 (GND), J314.B1 (GND), J314.B12 (GND), J314.S1 (SHIELD), R31.2, R32.2, R1.2
- net at J314.A4 (VBUS), J314.A9 (VBUS), J314.B4 (VBUS)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: now also D31.2 (A)
- new net: D1.1 (K), R1.1

Commit message: Added pull downs for safety
Parts:
- added R10, R15, R16, R17, R18, R19, R2, R20, R27, R28, R3, R4, R5, R6, R7, R8, R9: 10k, Capacitor_SMD:C_0603_1608Metric_Pad1.08x0.95mm_HandSolder, symbol Device:R
Connections:
- net +3.3V: now also R27.2
- net AUX_A: now also R9.2
- net AUX_B: now also R28.2
- net AUX_C: now also R20.2
- net AUX_D: now also R19.2
- net AUX_E: now also R18.2
- net AUX_F: now also R17.2
- net AUX_G: now also R16.2
- net AUX_H: now also R15.2
- net AUX_I: now also R10.2
- net GND: now also R10.1, R15.1, R16.1, R17.1, R18.1, R19.1, R2.1, R20.1, R28.1, R3.1, R4.1, R5.1, R6.1, R7.1, R8.1, R9.1
- net READY: now also R27.1
- net SPINDLE: now also R8.2
- net X_DIR: now also U32.13 (B7), R3.2; no longer U32.16 (B4)
- net X_DIR_3.3: now also U21.13 (2A2), U31.4 (GPIO3); no longer U21.8 (1A3), U31.6 (GPIO5)
- net X_STEP: now also U32.14 (B6), R4.2; no longer U32.17 (B3)
- net X_STEP_3.3: now also U21.15 (2A1), U31.1 (GPIO0); no longer U21.6 (1A2), U31.5 (GPIO4)
- net Y_DIR: now also U32.17 (B3), R7.2; no longer U32.13 (B7)
- net Y_DIR_3.3: now also U21.6 (1A2), U31.5 (GPIO4); no longer U21.13 (2A2), U31.4 (GPIO3)
- net Y_STEP: now also U32.15 (B5), R5.2; no longer U32.12 (B8)
- net Y_STEP_3.3: now also U21.17 (2A0), U31.2 (GPIO1); no longer U21.11 (2A3), U31.3 (GPIO2)
- net Z_DIR: now also U32.16 (B4), R6.2; no longer U32.15 (B5)
- net Z_DIR_3.3: now also U21.8 (1A3), U31.6 (GPIO5); no longer U21.17 (2A0), U31.2 (GPIO1)
- net Z_STEP: now also U32.12 (B8), R2.2; no longer U32.14 (B6)
- net Z_STEP_3.3: now also U21.11 (2A3), U31.3 (GPIO2); no longer U21.15 (2A1), U31.1 (GPIO0)
